Commit message: added maze.world

File: urdf/robotont_gazebo_common_lidar.urdf.xacro (robot description, xacro)
@@ -34,5 +34,6 @@
     </gazebo>
         <!-- Laser -->
-    <gazebo reference="hokuyo_link">
+    <gazebo reference="camera_link">
+    <!--<gazebo reference="hokuyo_link">-->
         <sensor type="ray" name="head_hokuyo_sensor">
             <pose>0 0 0 0 0 0</pose>
@@ -55,8 +56,4 @@
                 <noise>
                     <type>gaussian</type>
-                        <!-- Noise parameters based on published spec for Hokuyo laser
-                            achieving "+-30mm" accuracy at range < 10m.  A mean of 0.0m and
-                            stddev of 0.01m will put 99.7% of samples within 0.03m of the true
-                            reading. -->
                     <mean>0.0</mean>
                     <stddev>0.01</stddev>
@@ -65,5 +62,6 @@
             <plugin name="gazebo_ros_head_hokuyo_controller" filename="libgazebo_ros_laser.so">
                 <topicName>scan</topicName>
-                <frameName>hokuyo_link</frameName>
+                <frameName>camera_link</frameName>
+                <!-- <frameName>hokuyo_link</frameName>-->
             </plugin>
         </sensor>

File: urdf/robotont_gazebo_lidar.urdf.xacro (robot description, xacro)
@@ -30,5 +30,5 @@
         <origin xyz="-0.01 0 0.085" rpy="0 0 0"/>
     </joint>
-  <!-- Hokuyo Laser -->
+  <!-- Hokuyo Laser
     <joint name="hokuyo_joint" type="fixed">
         <axis xyz="0 1 0" />
@@ -47,5 +47,5 @@
             <origin xyz="0 0 0" rpy="0 0 0"/>
             <geometry>
-                <mesh filename="package://robotont_description/meshes/hokuyo.dae"/>
+                <mesh filename="package://robotont_gazebo/meshes/hokuyo.dae"/>
             </geometry>
         </visual>
@@ -56,3 +56,4 @@
         </inertial>
     </link>
+     -->
 </robot>
