Commit message: some changes

File: urdf/robotont_gazebo_common.urdf.xacro (robot description, xacro)
@@ -50,6 +50,6 @@
                     </clip>
                 </camera>
+-
                 <plugin name="kinect_camera_controller" filename="libgazebo_ros_openni_kinect.so">
-                    <robotNamespace>/</robotNamespace>
                     <cameraName>camera</cameraName>
                     <alwaysOn>true</alwaysOn>

File: urdf/robotont_gazebo_common_lidar.urdf.xacro (robot description, xacro)
@@ -64,5 +64,5 @@
             </ray>
             <plugin name="gazebo_ros_head_hokuyo_controller" filename="libgazebo_ros_laser.so">
-                <topicName>laser/scan</topicName>
+                <topicName>scan</topicName>
                 <frameName>hokuyo_link</frameName>
             </plugin>

File: urdf/robotont_gazebo_lidar.urdf.xacro (robot description, xacro)
@@ -2,5 +2,9 @@
 <robot xmlns:xacro="http://ros.org/wiki/xacro" name="robotont">
     <xacro:include filename="$(find robotont_description)/urdf/robotont_base.urdf.xacro"/>
+	<xacro:include filename="$(find robotont_gazebo)/urdf/_d435.urdf.xacro" />
 	<xacro:include filename="$(find robotont_gazebo)/urdf/robotont_gazebo_common_lidar.urdf.xacro" />
+    <xacro:sensor_d435 parent="${prefix}base_link">
+        <origin xyz="-0.12 0 0.21" rpy="0 0 0"/>
+    </xacro:sensor_d435>
     <!-- Computer -->
     <link name="${prefix}computer_link">

Commit message: cleaned up launch files and changed Robotont's colour

File: urdf/robotont_gazebo_common.urdf.xacro (robot description, xacro)
@@ -25,5 +25,5 @@
         <!-- Give materials to links -->
         <gazebo reference="${prefix}base_link">
-            <material>Robotont/BlueishTransparent</material>
+            <material>Gazebo/GreyTransparent </material>
         </gazebo>
         <gazebo reference="${prefix}camera_link">

Commit message: two descriptions; 3d_mapping should work now; colors.world for 3d_mapping

File: urdf/robotont_gazebo_common.urdf.xacro (robot description, xacro)
@@ -27,47 +27,49 @@
             <material>Gazebo/GreyTransparent </material>
         </gazebo>
-        <gazebo reference="${prefix}camera_link">
-            <material>Gazebo/Grey</material>
-        </gazebo>
         <gazebo reference="${prefix}computer_link">
             <material>Gazebo/Black</material>
         </gazebo>
-        <!-- Depth camera plugin -->
-        <gazebo reference="${prefix}camera_link">
-            <sensor type="depth" name="camera">
-                <always_on>true</always_on>
-                <update_rate>10.0</update_rate>
-                <camera>
-                    <horizontal_fov>${90.0*pi/180.0}</horizontal_fov>
-                    <image>
-                        <format>B8G8R8</format>
-                        <width>640</width>
-                        <height>480</height>
-                    </image>
-                    <clip>
-                        <near>0.02</near>
-                        <far>8.0</far>
-                    </clip>
-                </camera>
--
-                <plugin name="kinect_camera_controller" filename="libgazebo_ros_openni_kinect.so">
-                    <cameraName>camera</cameraName>
-                    <alwaysOn>true</alwaysOn>
-                    <updateRate>0.0</updateRate>
-                    <imageTopicName>color/image_raw</imageTopicName>
-                    <depthImageTopicName>depth/image_rect_raw</depthImageTopicName>
-                    <pointCloudTopicName>depth/points</pointCloudTopicName>
-                    <cameraInfoTopicName>color/camera_info</cameraInfoTopicName>
-                    <depthImageCameraInfoTopicName>depth/camera_info</depthImageCameraInfoTopicName>
-                    <frameName>camera_depth_optical_frame</frameName>
-                    <baseline>0.1</baseline>
-                    <distortion_k1>0.0</distortion_k1>
-                    <distortion_k2>0.0</distortion_k2>
-                    <distortion_k3>0.0</distortion_k3>
-                    <distortion_t1>0.0</distortion_t1>
-                    <distortion_t2>0.0</distortion_t2>
-                    <pointCloudCutoff>0.4</pointCloudCutoff>
-                </plugin>
-            </sensor>
-        </gazebo>
+        <!-- If nuc_desc then set true -->
+        <xacro:if value="$(arg add_cam)">
+            <gazebo reference="${prefix}camera_link">
+                <material>Gazebo/Grey</material>
+            </gazebo>
+            <!-- Depth camera plugin -->
+            <gazebo reference="${prefix}camera_link">
+                <sensor type="depth" name="camera">
+                    <always_on>true</always_on>
+                    <update_rate>10.0</update_rate>
+                    <camera>
+                        <horizontal_fov>${90.0*pi/180.0}</horizontal_fov>
+                        <image>
+                            <format>B8G8R8</format>
+                            <width>640</width>
+                            <height>480</height>
+                        </image>
+                        <clip>
+                            <near>0.02</near>
+                            <far>8.0</far>
+                        </clip>
+                    </camera>
+                    <plugin name="kinect_camera_controller" filename="libgazebo_ros_openni_kinect.so">
+                        <cameraName>camera</cameraName>
+                        <alwaysOn>true</alwaysOn>
+                        <updateRate>0.0</updateRate>
+                        <imageTopicName>color/image_raw</imageTopicName>
+                        <depthImageTopicName>depth/image_rect_raw</depthImageTopicName>
+                        <pointCloudTopicName>depth/points</pointCloudTopicName>
+                        <cameraInfoTopicName>color/camera_info</cameraInfoTopicName>
+                        <depthImageCameraInfoTopicName>depth/camera_info</depthImageCameraInfoTopicName>
+                        <frameName>camera_depth_optical_frame</frameName>
+                        <baseline>0.1</baseline>
+                        <distortion_k1>0.0</distortion_k1>
+                        <distortion_k2>0.0</distortion_k2>
+                        <distortion_k3>0.0</distortion_k3>
+                        <distortion_t1>0.0</distortion_t1>
+                        <distortion_t2>0.0</distortion_t2>
+                        <pointCloudCutoff>0.4</pointCloudCutoff>
+                    </plugin>
+                </sensor>
+            </gazebo>
+        </xacro:if>
 </robot>

Commit message: slight changes because camera assembly was separated from robotont_base

File: urdf/robotont_gazebo_common.urdf.xacro (robot description, xacro)
@@ -27,11 +27,17 @@
             <material>Gazebo/GreyTransparent </material>
         </gazebo>
+        <!-- If nuc_desc then set true -->'
         <gazebo reference="${prefix}computer_link">
             <material>Gazebo/Black</material>
         </gazebo>
-        <!-- If nuc_desc then set true -->
         <xacro:if value="$(arg add_cam)">
             <gazebo reference="${prefix}camera_link">
                 <material>Gazebo/Grey</material>
+            </gazebo>
+            <gazebo reference="${prefix}camera_assembly_link1">
+                <material>Gazebo/Grey</material>
+            </gazebo>
+            <gazebo reference="${prefix}camera_assembly_link2">
+                <material>Gazebo/GreyTransparent</material>
             </gazebo>
             <!-- Depth camera plugin -->

Commit message: gazebo_common is now common

File: urdf/robotont_gazebo_common.urdf.xacro (robot description, xacro)
@@ -1,81 +1,29 @@
 <?xml version="1.0"?>
 <robot xmlns:xacro="http://ros.org/wiki/xacro">
-        <xacro:include filename="$(find robotont_gazebo)/urdf/gazebo_rim.urdf.xacro"/>
-        <xacro:gazebo_rim_macro
-            name="back"
-            prefix="${prefix}"
-        />
-        <xacro:gazebo_rim_macro
-            name="right"
-            prefix="${prefix}"
-        />
-        <xacro:gazebo_rim_macro
-            name="left"
-            prefix="${prefix}"
-        />
-        <gazebo>
-            <plugin name="robotont_controller" filename="libgazebo_ros_planar_move.so">
-                <commandTopic>/robotont/cmd_vel</commandTopic>
-                <odometryTopic>/robotont/odom</odometryTopic>
-                <odometryFrame>odom</odometryFrame>
-                <odometryRate>30.0</odometryRate>
-                <robotBaseFrame>${prefix}base_footprint</robotBaseFrame>
-            </plugin>
-        </gazebo>
-        <!-- Give materials to links -->
-        <gazebo reference="${prefix}base_link">
-            <material>Gazebo/GreyTransparent </material>
-        </gazebo>
-        <!-- If nuc_desc then set true -->'
-        <gazebo reference="${prefix}computer_link">
-            <material>Gazebo/Black</material>
-        </gazebo>
-        <xacro:if value="$(arg add_cam)">
-            <gazebo reference="${prefix}camera_link">
-                <material>Gazebo/Grey</material>
-            </gazebo>
-            <gazebo reference="${prefix}camera_assembly_link1">
-                <material>Gazebo/Grey</material>
-            </gazebo>
-            <gazebo reference="${prefix}camera_assembly_link2">
-                <material>Gazebo/GreyTransparent</material>
-            </gazebo>
-            <!-- Depth camera plugin -->
-            <gazebo reference="${prefix}camera_link">
-                <sensor type="depth" name="camera">
-                    <always_on>true</always_on>
-                    <update_rate>10.0</update_rate>
-                    <camera>
-                        <horizontal_fov>${90.0*pi/180.0}</horizontal_fov>
-                        <image>
-                            <format>B8G8R8</format>
-                            <width>640</width>
-                            <height>480</height>
-                        </image>
-                        <clip>
-                            <near>0.02</near>
-                            <far>8.0</far>
-                        </clip>
-                    </camera>
-                    <plugin name="kinect_camera_controller" filename="libgazebo_ros_openni_kinect.so">
-                        <cameraName>camera</cameraName>
-                        <alwaysOn>true</alwaysOn>
-                        <updateRate>0.0</updateRate>
-                        <imageTopicName>color/image_raw</imageTopicName>
-                        <depthImageTopicName>depth/image_rect_raw</depthImageTopicName>
-                        <pointCloudTopicName>depth/points</pointCloudTopicName>
-                        <cameraInfoTopicName>color/camera_info</cameraInfoTopicName>
-                        <depthImageCameraInfoTopicName>depth/camera_info</depthImageCameraInfoTopicName>
-                        <frameName>camera_depth_optical_frame</frameName>
-                        <baseline>0.1</baseline>
-                        <distortion_k1>0.0</distortion_k1>
-                        <distortion_k2>0.0</distortion_k2>
-                        <distortion_k3>0.0</distortion_k3>
-                        <distortion_t1>0.0</distortion_t1>
-                        <distortion_t2>0.0</distortion_t2>
-                        <pointCloudCutoff>0.4</pointCloudCutoff>
-                    </plugin>
-                </sensor>
-            </gazebo>
-        </xacro:if>
+    <xacro:include filename="$(find robotont_gazebo)/urdf/gazebo_rim.urdf.xacro"/>
+    <xacro:gazebo_rim_macro
+        name="back"
+        prefix="${prefix}"
+    />
+    <xacro:gazebo_rim_macro
+        name="right"
+        prefix="${prefix}"
+    />
+    <xacro:gazebo_rim_macro
+        name="left"
+        prefix="${prefix}"
+    />
+    <gazebo>
+        <plugin name="robotont_controller" filename="libgazebo_ros_planar_move.so">
+            <commandTopic>/robotont/cmd_vel</commandTopic>
+            <odometryTopic>/robotont/odom</odometryTopic>
+            <odometryFrame>odom</odometryFrame>
+            <odometryRate>30.0</odometryRate>
+            <robotBaseFrame>${prefix}base_footprint</robotBaseFrame>
+        </plugin>
+    </gazebo>
+    <!-- Give materials to links -->
+    <gazebo reference="${prefix}base_link">
+        <material>Gazebo/GreyTransparent </material>
+    </gazebo>
 </robot>

File: urdf/robotont_gazebo_lidar.urdf.xacro (robot description, xacro)
@@ -2,6 +2,4 @@
 <robot xmlns:xacro="http://ros.org/wiki/xacro" name="robotont">
     <xacro:include filename="$(find robotont_description)/urdf/robotont_base.urdf.xacro"/>
-    <xacro:include ns="robotont" filename="$(find robotont_gazebo)/urdf/gazebo_lidar.urdf.xacro"/>
-    <xacro:arg name="add_cam" default="false"/>
 	<xacro:include filename="$(find robotont_gazebo)/urdf/robotont_gazebo_common.urdf.xacro" />
     <!-- Computer -->
@@ -54,3 +52,40 @@
         </inertial>
     </link>
+    <gazebo reference="${prefix}computer_link">
+        <material>Gazebo/Black</material>
+    </gazebo>
+    <gazebo reference="${prefix}camera_link">
+        <material>Gazebo/Grey</material>
+    </gazebo>
+    <gazebo reference="hokuyo_link">
+        <sensor type="ray" name="head_hokuyo_sensor">
+            <pose>0 0 0 0 0 0</pose>
+            <visualize>false</visualize>
+            <update_rate>40</update_rate>
+            <ray>
+                <scan>
+                    <horizontal>
+                        <samples>720</samples>
+                        <resolution>1</resolution>
+                        <min_angle>-3.14159</min_angle>
+                        <max_angle>3.14159</max_angle>
+                    </horizontal>
+                </scan>
+                <range>
+                    <min>0.10</min>
+                    <max>30.0</max>
+                    <resolution>0.01</resolution>
+                </range>
+                <noise>
+                    <type>gaussian</type>
+                    <mean>0.0</mean>
+                    <stddev>0.01</stddev>
+                </noise>
+            </ray>
+            <plugin name="gazebo_ros_head_hokuyo_controller" filename="libgazebo_ros_laser.so">
+                <topicName>scan</topicName>
+                <frameName>hokuyo_link</frameName>
+            </plugin>
+        </sensor>
+    </gazebo>
 </robot>

File: urdf/robotont_gazebo_nuc.urdf.xacro (robot description, xacro)
@@ -3,5 +3,53 @@
     <xacro:arg name= "simulated" default="true" />
     <xacro:include filename="$(find robotont_nuc_description)/urdf/robotont_realsense.urdf.xacro"/>
-    <xacro:arg name="add_cam" default="true"/>
 	<xacro:include filename="$(find robotont_gazebo)/urdf/robotont_gazebo_common.urdf.xacro" />
+    <gazebo reference="${prefix}computer_link">
+        <material>Gazebo/Black</material>
+    </gazebo>
+    <gazebo reference="${prefix}camera_link">
+        <material>Gazebo/Grey</material>
+    </gazebo>
+    <gazebo reference="${prefix}camera_assembly_link1">
+        <material>Gazebo/Grey</material>
+    </gazebo>
+    <gazebo reference="${prefix}camera_assembly_link2">
+        <material>Gazebo/GreyTransparent</material>
+    </gazebo>
+    <!-- Depth camera plugin -->
+    <gazebo reference="${prefix}camera_link">
+        <sensor type="depth" name="camera">
+            <always_on>true</always_on>
+            <update_rate>10.0</update_rate>
+            <camera>
+                <horizontal_fov>${90.0*pi/180.0}</horizontal_fov>
+                <image>
+                    <format>B8G8R8</format>
+                    <width>640</width>
+                    <height>480</height>
+                </image>
+                <clip>
+                    <near>0.02</near>
+                    <far>8.0</far>
+                </clip>
+            </camera>
+            <plugin name="kinect_camera_controller" filename="libgazebo_ros_openni_kinect.so">
+                <cameraName>camera</cameraName>
+                <alwaysOn>true</alwaysOn>
+                <updateRate>0.0</updateRate>
+                <imageTopicName>color/image_raw</imageTopicName>
+                <depthImageTopicName>depth/image_rect_raw</depthImageTopicName>
+                <pointCloudTopicName>depth/points</pointCloudTopicName>
+                <cameraInfoTopicName>color/camera_info</cameraInfoTopicName>
+                <depthImageCameraInfoTopicName>depth/camera_info</depthImageCameraInfoTopicName>
+                <frameName>camera_depth_optical_frame</frameName>
+                <baseline>0.1</baseline>
+                <distortion_k1>0.0</distortion_k1>
+                <distortion_k2>0.0</distortion_k2>
+                <distortion_k3>0.0</distortion_k3>
+                <distortion_t1>0.0</distortion_t1>
+                <distortion_t2>0.0</distortion_t2>
+                <pointCloudCutoff>0.4</pointCloudCutoff>
+            </plugin>
+        </sensor>
+    </gazebo>
 </robot>
