Commit message: semi-broken

File: urdf/robotont_gazebo_basic.urdf.xacro (robot description, xacro)
@@ -1,4 +1,6 @@
 <?xml version="1.0"?>
 <robot xmlns:xacro="http://ros.org/wiki/xacro" name="robotont">
+    <xacro:arg name="__ns" default=""/>
+    <xacro:property name= "__ns" value="$(arg __ns)"/>
     <xacro:include filename="$(find robotont_description)/urdf/robotont_base.urdf.xacro"/>
 	<xacro:include filename="$(find robotont_gazebo)/urdf/robotont_gazebo_common.urdf.xacro" />

File: urdf/robotont_gazebo_common.urdf.xacro (robot description, xacro)
@@ -16,7 +16,7 @@
     <gazebo>
         <plugin name="robotont_controller" filename="libgazebo_ros_planar_move.so">
-            <commandTopic>/cmd_vel</commandTopic>
-            <odometryTopic>/odom</odometryTopic>
-            <odometryFrame>odom</odometryFrame>
+            <commandTopic>${__ns}/cmd_vel</commandTopic>
+            <odometryTopic>${__ns}/odom</odometryTopic>
+            <odometryFrame>${prefix}odom</odometryFrame>
             <odometryRate>30.0</odometryRate>
             <robotBaseFrame>${prefix}base_footprint</robotBaseFrame>

File: urdf/robotont_gazebo_lidar.urdf.xacro (robot description, xacro)
@@ -1,4 +1,6 @@
 <?xml version="1.0"?>
 <robot xmlns:xacro="http://ros.org/wiki/xacro" name="robotont">
+    <xacro:arg name="__ns" default=""/>
+    <xacro:property name= "__ns" value="$(arg __ns)"/>
     <xacro:include filename="$(find robotont_description)/urdf/robotont_base.urdf.xacro"/>
 	<xacro:include filename="$(find robotont_gazebo)/urdf/robotont_gazebo_common.urdf.xacro" />
@@ -27,5 +29,5 @@
     </joint>
     <!-- Hokuyo Laser -->
-    <joint name="hokuyo_joint" type="fixed">
+    <joint name="{prefix}hokuyo_joint" type="fixed">
         <axis xyz="0 1 0" />
         <origin xyz="0 0 0.05" rpy="0 0 0"/>
@@ -33,5 +35,5 @@
         <child link="hokuyo_link"/>
     </joint>
-    <link name="hokuyo_link">
+    <link name="{prefix}hokuyo_link">
         <collision>
             <origin xyz="0 0 0" rpy="0 0 0"/>
@@ -84,6 +86,6 @@
             </ray>
             <plugin name="gazebo_ros_head_hokuyo_controller" filename="libgazebo_ros_laser.so">
-                <topicName>scan</topicName>
-                <frameName>hokuyo_link</frameName>
+                <topicName>{__ns}/scan</topicName>
+                <frameName>{prefix}hokuyo_link</frameName>
             </plugin>
         </sensor>

File: urdf/robotont_gazebo_nuc.urdf.xacro (robot description, xacro)
@@ -1,4 +1,6 @@
 <?xml version="1.0"?>
 <robot xmlns:xacro="http://ros.org/wiki/xacro" name="robotont">
+    <xacro:arg name="__ns" default=""/>
+    <xacro:property name= "__ns" value="$(arg __ns)"/>
     <xacro:arg name= "simulated" default="true" />
     <xacro:include filename="$(find robotont_nuc_description)/urdf/robotont_realsense.urdf.xacro"/>
@@ -20,11 +22,11 @@
         <sensor type="depth" name="camera">
             <always_on>true</always_on>
-            <update_rate>10.0</update_rate>
+            <update_rate>30.0</update_rate>
             <camera>
                 <horizontal_fov>${90.0*pi/180.0}</horizontal_fov>
                 <image>
                     <format>B8G8R8</format>
-                    <width>640</width>
-                    <height>480</height>
+                    <width>1280</width>
+                    <height>720</height>
                 </image>
                 <clip>
@@ -34,5 +36,5 @@
             </camera>
             <plugin name="kinect_camera_controller" filename="libgazebo_ros_openni_kinect.so">
-                <cameraName>camera</cameraName>
+                <cameraName>${__ns}/camera</cameraName>
                 <alwaysOn>true</alwaysOn>
                 <updateRate>0.0</updateRate>
@@ -42,5 +44,5 @@
                 <cameraInfoTopicName>color/camera_info</cameraInfoTopicName>
                 <depthImageCameraInfoTopicName>depth/camera_info</depthImageCameraInfoTopicName>
-                <frameName>camera_depth_optical_frame</frameName>
+                <frameName>${prefix}camera_depth_optical_frame</frameName>
                 <baseline>0.1</baseline>
                 <distortion_k1>0.0</distortion_k1>

Commit message: fixes in ns

File: urdf/robotont_gazebo_basic.urdf.xacro (robot description, xacro)
@@ -1,6 +1,4 @@
 <?xml version="1.0"?>
 <robot xmlns:xacro="http://ros.org/wiki/xacro" name="robotont">
-    <xacro:arg name="__ns" default=""/>
-    <xacro:property name= "__ns" value="$(arg __ns)"/>
     <xacro:include filename="$(find robotont_description)/urdf/robotont_base.urdf.xacro"/>
 	<xacro:include filename="$(find robotont_gazebo)/urdf/robotont_gazebo_common.urdf.xacro" />

File: urdf/robotont_gazebo_common.urdf.xacro (robot description, xacro)
@@ -16,6 +16,6 @@
     <gazebo>
         <plugin name="robotont_controller" filename="libgazebo_ros_planar_move.so">
-            <commandTopic>${__ns}/cmd_vel</commandTopic>
-            <odometryTopic>${__ns}/odom</odometryTopic>
+            <commandTopic>cmd_vel</commandTopic>
+            <odometryTopic>odom</odometryTopic>
             <odometryFrame>${prefix}odom</odometryFrame>
             <odometryRate>30.0</odometryRate>

File: urdf/robotont_gazebo_lidar.urdf.xacro (robot description, xacro)
@@ -1,6 +1,4 @@
 <?xml version="1.0"?>
 <robot xmlns:xacro="http://ros.org/wiki/xacro" name="robotont">
-    <xacro:arg name="__ns" default=""/>
-    <xacro:property name= "__ns" value="$(arg __ns)"/>
     <xacro:include filename="$(find robotont_description)/urdf/robotont_base.urdf.xacro"/>
 	<xacro:include filename="$(find robotont_gazebo)/urdf/robotont_gazebo_common.urdf.xacro" />
@@ -86,5 +84,5 @@
             </ray>
             <plugin name="gazebo_ros_head_hokuyo_controller" filename="libgazebo_ros_laser.so">
-                <topicName>${__ns}/scan</topicName>
+                <topicName>scan</topicName>
                 <frameName>${prefix}hokuyo_link</frameName>
             </plugin>

File: urdf/robotont_gazebo_nuc.urdf.xacro (robot description, xacro)
@@ -1,6 +1,4 @@
 <?xml version="1.0"?>
 <robot xmlns:xacro="http://ros.org/wiki/xacro" name="robotont">
-    <xacro:arg name="__ns" default=""/>
-    <xacro:property name= "__ns" value="$(arg __ns)"/>
     <xacro:arg name= "simulated" default="true" />
     <xacro:include filename="$(find robotont_nuc_description)/urdf/robotont_realsense.urdf.xacro"/>
@@ -36,5 +34,5 @@
             </camera>
             <plugin name="kinect_camera_controller" filename="libgazebo_ros_openni_kinect.so">
-                <cameraName>${__ns}/camera</cameraName>
+                <cameraName>camera</cameraName>
                 <alwaysOn>true</alwaysOn>
                 <updateRate>0.0</updateRate>
